File: mdrpcb/mdrpcb.kicad_sch (KiCad schematic)
At the start: 38 parts, among them J1 Conn_02x04_Odd_Even, J10 Conn_01x06, J11 Conn_01x06, J2 Conn_01x03, J3 SM04B-SRSS-TB, J4 Conn_01x03, J5 Conn_01x03, J6 Conn_01x03, J7 Conn_01x03, J8 Conn_01x03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

Commit message: Add files via upload
Parts:
- added C5: 100nF, Capacitor_THT:CP_Radial_D4.0mm_P1.50mm, symbol Device:C
- added R12: 100, Resistor_THT:R_Axial_DIN0204_L3.6mm_D1.6mm_P1.90mm_Vertical, symbol Device:R
- added R13: 10k, Resistor_THT:R_Axial_DIN0204_L3.6mm_D1.6mm_P1.90mm_Vertical, symbol Device:R
- added SW5: SW_Push, Button_Switch_THT:SW_PUSH_6mm, symbol Switch:SW_Push
Connections:
- net +3V3: now also R13.1
- net GND: now also C5.2, R12.2
- net SW2: now also C5.1, R13.2, SW5.2
- new net: R12.1, SW5.1
Other:
- note added: "Bonus Switch (lol)"
- note added: "Switch 3"
- moved on the sheet: J10, J11, J5, J6, J7, J8, J9

Commit message: Add files via upload
Other:
- note added: "SPI0"
- note added: "SPI1"
- note removed: "UART0"
- note removed: "UART1"
Changed lines of the file:
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@@
     (effects (font (size 1.27 1.27)) (justify left bottom))
   )
-  (text "UART1" (at 187.96 125.73 0)
+  (text "SPI1" (at 187.96 125.73 0)
     (effects (font (size 1.27 1.27)) (justify left bottom))
   )
@@
     (effects (font (size 1.27 1.27)) (justify left bottom))
   )
-  (text "UART0" (at 166.37 125.73 0)
+  (text "SPI0" (at 166.37 125.73 0)
     (effects (font (size 1.27 1.27)) (justify left bottom))
   )
