File: fprpcb/fprpcb.kicad_sch (KiCad schematic)
At the start: 49 parts, among them J1 Conn_02x04_Odd_Even, J2 Conn_01x02, J3 Conn_01x03, J4 Conn_01x03, J5 Conn_01x03, J6 Conn_01x03, J7 Conn_01x06, J8 Conn_01x04, SW1 Conn_01x02_Pin, SW2 Conn_01x02_Pin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

Commit message: updated fprpcb
Parts:
- removed C8: 100nF, Capacitor_THT:CP_Radial_D4.0mm_P1.50mm, symbol Device:C
- removed R16: 100, Resistor_THT:R_Axial_DIN0204_L3.6mm_D1.6mm_P5.08mm_Horizontal, symbol Device:R
- removed R17: 10k, Resistor_THT:R_Axial_DIN0204_L3.6mm_D1.6mm_P5.08mm_Horizontal, symbol Device:R
Connections:
- net +3.3V: no longer SW6.1 (Pin_1)
- net B+: now also SW6.2 (Pin_2)
- new net VSYS: SW6.1 (Pin_1)
Changed lines of the file:
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@@
   (junction (at 198.12 153.67) (diameter 0) (color 0 0 0 0)
   )
-  (junction (at 201.93 108.585) (diameter 0) (color 0 0 0 0)
-  )
   (junction (at 243.84 153.67) (diameter 0) (color 0 0 0 0)
   )
@@
   (junction (at 198.12 135.89) (diameter 0) (color 0 0 0 0)
   )
-  (junction (at 201.93 90.805) (diameter 0) (color 0 0 0 0)
-  )
   (junction (at 93.98 184.15) (diameter 0) (color 0 0 0 0)
   )
@@
     (stroke (width 0) (type default))
   )
-  (wire (pts (xy 201.93 88.265) (xy 201.93 90.805))
-    (stroke (width 0) (type default))
-  )
   (wire (pts (xy 137.16 135.89) (xy 137.16 137.16))
     (stroke (width 0) (type default))
@@
     (stroke (width 0) (type default))
   )
-  (wire (pts (xy 201.93 98.425) (xy 201.93 108.585))
-    (stroke (width 0) (type default))
-  )
   (wire (pts (xy 257.81 34.29) (xy 261.62 34.29))
     (stroke (width 0) (type default))
@@
     (stroke (width 0) (type default))
   )
-  (wire (pts (xy 189.23 108.585) (xy 201.93 108.585))
-    (stroke (width 0) (type default))
-  )
   (wire (pts (xy 88.265 70.485) (xy 93.345 70.485))
     (stroke (width 0) (type default))
@@
     (stroke (width 0) (type default))
   )
-  (wire (pts (xy 201.93 90.805) (xy 208.28 90.805))
-    (stroke (width 0) (type default))
-  )
   (wire (pts (xy 88.265 40.005) (xy 93.345 40.005))
     (stroke (width 0) (type default))
@@
     (stroke (width 0) (type default))
   )
-  (wire (pts (xy 201.93 111.76) (xy 201.93 108.585))
-    (stroke (width 0) (type default))
-  )
   (wire (pts (xy 88.265 42.545) (xy 97.155 42.545))
     (stroke (width 0) (type default))
@@
     (effects (font (size 1.27 1.27)) (justify left bottom))
   )
+  (label "B+" (at 189.23 100.965 0) (fields_autoplaced)
+    (effects (font (size 1.27 1.27)) (justify left bottom))
+  )
   (label "GP1_UART0_RX" (at 31.115 50.165 180) (fields_autoplaced)
     (effects (font (size 1.27 1.27)) (justify right bottom))
@@
     (effects (font (size 1.27 1.27)) (justify left bottom))
   )
+  (label "VSYS" (at 201.93 90.805 0) (fields_autoplaced)
+    (effects (font (size 1.27 1.27)) (justify left bottom))
+  )
   (label "GP6_INT" (at 160.655 139.7 270) (fields_autoplaced)
     (effects (font (size 1.27 1.27)) (justify right bottom))
@@
     (effects (font (size 1.27 1.27)) (justify left bottom))
   )
-  (label "+3.3V" (at 208.28 90.805 0) (fields_autoplaced)
-    (effects (font (size 1.27 1.27)) (justify left bottom))
-  )
   (label "GP0_UART0_TX" (at 31.115 47.625 180) (fields_autoplaced)
     (effects (font (size 1.27 1.27)) (justify right bottom))
@@
     )
   )
-  (symbol (lib_id "Device:R") (at 189.23 104.775 0) (unit 1)
-    (in_bom yes) (on_board yes) (dnp no) (fields_autoplaced)
-    (property "Reference" "R16" (at 191.77 103.505 0)
-      (effects (font (size 1.27 1.27)) (justify left))
-    )
-    (property "Value" "100" (at 191.77 106.045 0)
-      (effects (font (size 1.27 1.27)) (justify left))
-    )
-    (property "Footprint" "Resistor_THT:R_Axial_DIN0204_L3.6mm_D1.6mm_P5.08mm_Horizontal" (at 187.452 104.775 90)
-      (effects (font (size 1.27 1.27)) hide)
-    )
-    (property "Datasheet" "~" (at 189.23 104.775 0)
-      (effects (font (size 1.27 1.27)) hide)
-    )
-    (pin "1")
-    (pin "2")
-    (instances
-      (project "fprpcb"
-        (path "/256b697e-9752-4e3a-a338-bc05701ab36e"
-          (reference "R16") (unit 1)
-        )
-      )
-    )
-  )
   (symbol (lib_id "power:GND") (at 198.12 153.67 0) (unit 1)
     (in_bom yes) (on_board yes) (dnp no) (fields_autoplaced)
@@
     )
   )
-  (symbol (lib_id "power:+3V3") (at 201.93 80.645 0) (unit 1)
-    (in_bom yes) (on_board yes) (dnp no) (fields_autoplaced)
-    (property "Reference" "#PWR016" (at 201.93 84.455 0)
-      (effects (font (size 1.27 1.27)) hide)
-    )
-    (property "Value" "+3V3" (at 201.93 76.835 0)
-      (effects (font (size 1.27 1.27)))
-    )
-    (property "Footprint" "" (at 201.93 80.645 0)
-      (effects (font (size 1.27 1.27)) hide)
-    )
-    (property "Datasheet" "" (at 201.93 80.645 0)
-      (effects (font (size 1.27 1.27)) hide)
-    )
-    (pin "1")
-    (instances
-      (project "fprpcb"
-        (path "/256b697e-9752-4e3a-a338-bc05701ab36e"
-          (reference "#PWR016") (unit 1)
-        )
-      )
-    )
-  )
   (symbol (lib_id "power:VBUS") (at 144.145 32.385 90) (unit 1)
     (in_bom yes) (on_board yes) (dnp no) (fields_autoplaced)
@@
     )
   )
-  (symbol (lib_id "Device:C") (at 201.93 94.615 0) (unit 1)
-    (in_bom yes) (on_board yes) (dnp no) (fields_autoplaced)
-    (property "Reference" "C8" (at 205.74 93.345 0)
-      (effects (font (size 1.27 1.27)) (justify left))
-    )
-    (property "Value" "100nF" (at 205.74 95.885 0)
-      (effects (font (size 1.27 1.27)) (justify left))
-    )
-    (property "Footprint" "Capacitor_THT:CP_Radial_D4.0mm_P1.50mm" (at 202.8952 98.425 0)
-      (effects (font (size 1.27 1.27)) hide)
-    )
-    (property "Datasheet" "~" (at 201.93 94.615 0)
-      (effects (font (size 1.27 1.27)) hide)
-    )
-    (pin "1")
-    (pin "2")
-    (instances
-      (project "fprpcb"
-        (path "/256b697e-9752-4e3a-a338-bc05701ab36e"
-          (reference "C8") (unit 1)
-        )
-      )
-    )
-  )
   (symbol (lib_id "Device:R") (at 231.14 149.86 0) (unit 1)
     (in_bom yes) (on_board yes) (dnp no) (fields_autoplaced)
@@
       (effects (font (size 1.27 1.27)) hide)
     )
-    (property "Value" "+5V" (at 160.655 34.925 90)
+    (property "Value" "VSYS" (at 160.02 35.56 90)
       (effects (font (size 1.27 1.27)) (justify left))
     )
@@
     )
   )
-  (symbol (lib_id "Device:R") (at 201.93 84.455 0) (unit 1)
-    (in_bom yes) (on_board yes) (dnp no) (fields_autoplaced)
-    (property "Reference" "R17" (at 204.47 83.185 0)
-      (effects (font (size 1.27 1.27)) (justify left))
-    )
-    (property "Value" "10k" (at 204.47 85.725 0)
-      (effects (font (size 1.27 1.27)) (justify left))
-    )
-    (property "Footprint" "Resistor_THT:R_Axial_DIN0204_L3.6mm_D1.6mm_P5.08mm_Horizontal" (at 200.152 84.455 90)
-      (effects (font (size 1.27 1.27)) hide)
-    )
-    (property "Datasheet" "~" (at 201.93 84.455 0)
-      (effects (font (size 1.27 1.27)) hide)
-    )
-    (pin "1")
-    (pin "2")
-    (instances
-      (project "fprpcb"
-        (path "/256b697e-9752-4e3a-a338-bc05701ab36e"
-          (reference "R17") (unit 1)
-        )
-      )
-    )
-  )
   (symbol (lib_id "Device:R") (at 260.35 106.68 0) (unit 1)
     (in_bom yes) (on_board yes) (dnp no) (fields_autoplaced)
@@
         )
       )
-    )
-  )
-  (symbol (lib_id "power:GND") (at 201.93 111.76 0) (unit 1)
-    (in_bom yes) (on_board yes) (dnp no) (fields_autoplaced)
-    (property "Reference" "#PWR035" (at 201.93 118.11 0)
-      (effects (font (size 1.27 1.27)) hide)
-    )
-    (property "Value" "GND" (at 201.93 116.84 0)
-      (effects (font (size 1.27 1.27)))
-    )
-    (property "Footprint" "" (at 201.93 111.76 0)
-      (effects (font (size 1.27 1.27)) hide)
-    )
-    (property "Datasheet" "" (at 201.93 111.76 0)
-      (effects (font (size 1.27 1.27)) hide)
-    )
-    (pin "1")
-    (instances
-      (project "fprpcb"
-        (path "/256b697e-9752-4e3a-a338-bc05701ab36e"
-          (reference "#PWR035") (unit 1)
-        )
-      )

Commit message: fixed power switch issue where ghost components were showing up on the board
Connections:
- net VSYS is gone; now on net +5V: SW6.1 (Pin_1)
Changed lines of the file:
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@@
   (junction (at 243.84 135.89) (diameter 0) (color 0 0 0 0)
+  )
+  (junction (at 88.9 29.845) (diameter 0) (color 0 0 0 0)
   )
   (junction (at 187.325 31.75) (diameter 0) (color 0 0 0 0)
@@
     (stroke (width 0) (type default))
   )
+  (wire (pts (xy 92.075 31.75) (xy 88.9 31.75))
+    (stroke (width 0) (type default))
+  )
   (wire (pts (xy 31.115 60.325) (xy 37.465 60.325))
     (stroke (width 0) (type default))
@@
     (stroke (width 0) (type default))
   )
+  (wire (pts (xy 88.9 31.75) (xy 88.9 29.845))
+    (stroke (width 0) (type default))
+  )
   (wire (pts (xy 187.325 26.67) (xy 187.96 26.67))
     (stroke (width 0) (type default))
@@
     (stroke (width 0) (type default))
   )
+  (wire (pts (xy 88.9 29.845) (xy 95.885 29.845))
+    (stroke (width 0) (type default))
+  )
   (wire (pts (xy 273.05 90.17) (xy 273.05 92.71))
     (stroke (width 0) (type default))
@@
     (stroke (width 0) (type default))
   )
-  (wire (pts (xy 88.265 29.845) (xy 95.885 29.845))
+  (wire (pts (xy 88.265 29.845) (xy 88.9 29.845))
     (stroke (width 0) (type default))
   )
@@
     (effects (font (size 1.27 1.27)) (justify left bottom))
   )
+  (label "VSYS" (at 92.075 31.75 0) (fields_autoplaced)
+    (effects (font (size 1.27 1.27)) (justify left bottom))
+  )

Commit message: fprpcb
Connections:
- net +5V: now also SW6.2 (Pin_2)
- net B+: no longer SW6.2 (Pin_2)
Changed lines of the file:
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@@
+    (stroke (width 0) (type default))
+  )
+  (wire (pts (xy 193.675 100.965) (xy 193.675 100.33))
     (stroke (width 0) (type default))
   )
@@
   )
   (wire (pts (xy 198.12 143.51) (xy 198.12 153.67))
+    (stroke (width 0) (type default))
+  )
+  (wire (pts (xy 189.23 100.965) (xy 193.675 100.965))
     (stroke (width 0) (type default))
   )
@@
     (effects (font (size 1.27 1.27)) (justify left bottom))
   )
-  (label "B+" (at 189.23 100.965 0) (fields_autoplaced)
-    (effects (font (size 1.27 1.27)) (justify left bottom))
-  )
   (label "GP1_UART0_RX" (at 31.115 50.165 180) (fields_autoplaced)
     (effects (font (size 1.27 1.27)) (justify right bottom))
@@
     (effects (font (size 1.27 1.27)) (justify left bottom))
   )
+  (label "VSYS" (at 257.81 20.32 0) (fields_autoplaced)
+    (effects (font (size 1.27 1.27)) (justify left bottom))
+  )
   (label "SWDIO" (at 97.155 42.545 0) (fields_autoplaced)
     (effects (font (size 1.27 1.27)) (justify left bottom))
@@
     (effects (font (size 1.27 1.27)) (justify left bottom))
   )
+  (label "VSYS" (at 144.78 137.16 270) (fields_autoplaced)
+    (effects (font (size 1.27 1.27)) (justify right bottom))
+  )
   (label "SPI0_SCK" (at 137.16 135.89 270) (fields_autoplaced)
     (effects (font (size 1.27 1.27)) (justify right bottom))
@@
     (effects (font (size 1.27 1.27)) (justify right bottom))
   )
+  (label "Out+" (at 193.675 100.33 0) (fields_autoplaced)
+    (effects (font (size 1.27 1.27)) (justify left bottom))
+  )
   (label "SW2" (at 97.155 55.245 0) (fields_autoplaced)
     (effects (font (size 1.27 1.27)) (justify left bottom))
@@
   )
   (label "GND" (at 208.28 35.56 0) (fields_autoplaced)
+    (effects (font (size 1.27 1.27)) (justify left bottom))
+  )
+  (label "Out+" (at 250.825 21.59 0) (fields_autoplaced)
     (effects (font (size 1.27 1.27)) (justify left bottom))
   )
@@
     )
   )
-  (symbol (lib_id "power:+5V") (at 144.78 137.16 180) (unit 1)
-    (in_bom yes) (on_board yes) (dnp no) (fields_autoplaced)
-    (property "Reference" "#PWR045" (at 144.78 133.35 0)
-      (effects (font (size 1.27 1.27)) hide)
-    )
-    (property "Value" "+5V" (at 144.78 142.24 0)
-      (effects (font (size 1.27 1.27)))
-    )
-    (property "Footprint" "" (at 144.78 137.16 0)
-      (effects (font (size 1.27 1.27)) hide)
-    )
-    (property "Datasheet" "" (at 144.78 137.16 0)
-      (effects (font (size 1.27 1.27)) hide)
-    )
-    (pin "1")
-    (instances
-      (project "fprpcb"
-        (path "/256b697e-9752-4e3a-a338-bc05701ab36e"
-          (reference "#PWR045") (unit 1)
-        )
-      )
-    )
-  )
   (symbol (lib_id "power:+3V3") (at 242.57 82.55 0) (unit 1)
     (in_bom yes) (on_board yes) (dnp no) (fields_autoplaced)
@@
         )
       )
-    )
-  )
-  (symbol (lib_id "power:+5V") (at 257.81 20.32 0) (unit 1)
-    (in_bom yes) (on_board yes) (dnp no)
-    (property "Reference" "#PWR032" (at 257.81 24.13 0)
-      (effects (font (size 1.27 1.27)) hide)
-    )
-    (property "Value" "VSYS" (at 258.445 17.145 0)
-      (effects (font (size 1.27 1.27)) (justify left))
-    )
-    (property "Footprint" "" (at 257.81 20.32 0)
-      (effects (font (size 1.27 1.27)) hide)
-    )
-    (property "Datasheet" "" (at 257.81 20.32 0)
-      (effects (font (size 1.27 1.27)) hide)
-    )
-    (pin "1")
-    (instances
-      (project "fprpcb"
-        (path "/256b697e-9752-4e3a-a338-bc05701ab36e"
-          (reference "#PWR032") (unit 1)
-        )
-      )

Commit message: Revert "fprpcb"
This reverts commit a24959e1a84143555ed98c59d3b6709d6d6878c6.
Connections:
- net +5V: no longer SW6.2 (Pin_2)
- net B+: now also SW6.2 (Pin_2)
Changed lines of the file:
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@@
-    (stroke (width 0) (type default))
-  )
-  (wire (pts (xy 193.675 100.965) (xy 193.675 100.33))
     (stroke (width 0) (type default))
   )
@@
   )
   (wire (pts (xy 198.12 143.51) (xy 198.12 153.67))
-    (stroke (width 0) (type default))
-  )
-  (wire (pts (xy 189.23 100.965) (xy 193.675 100.965))
     (stroke (width 0) (type default))
   )
@@
     (effects (font (size 1.27 1.27)) (justify left bottom))
   )
+  (label "B+" (at 189.23 100.965 0) (fields_autoplaced)
+    (effects (font (size 1.27 1.27)) (justify left bottom))
+  )
   (label "GP1_UART0_RX" (at 31.115 50.165 180) (fields_autoplaced)
     (effects (font (size 1.27 1.27)) (justify right bottom))
@@
     (effects (font (size 1.27 1.27)) (justify left bottom))
   )
-  (label "VSYS" (at 257.81 20.32 0) (fields_autoplaced)
-    (effects (font (size 1.27 1.27)) (justify left bottom))
-  )
   (label "SWDIO" (at 97.155 42.545 0) (fields_autoplaced)
     (effects (font (size 1.27 1.27)) (justify left bottom))
@@
     (effects (font (size 1.27 1.27)) (justify left bottom))
   )
-  (label "VSYS" (at 144.78 137.16 270) (fields_autoplaced)
-    (effects (font (size 1.27 1.27)) (justify right bottom))
-  )
   (label "SPI0_SCK" (at 137.16 135.89 270) (fields_autoplaced)
     (effects (font (size 1.27 1.27)) (justify right bottom))
@@
     (effects (font (size 1.27 1.27)) (justify right bottom))
   )
-  (label "Out+" (at 193.675 100.33 0) (fields_autoplaced)
-    (effects (font (size 1.27 1.27)) (justify left bottom))
-  )
   (label "SW2" (at 97.155 55.245 0) (fields_autoplaced)
     (effects (font (size 1.27 1.27)) (justify left bottom))
@@
   )
   (label "GND" (at 208.28 35.56 0) (fields_autoplaced)
-    (effects (font (size 1.27 1.27)) (justify left bottom))
-  )
-  (label "Out+" (at 250.825 21.59 0) (fields_autoplaced)
     (effects (font (size 1.27 1.27)) (justify left bottom))
   )
@@
     )
   )
+  (symbol (lib_id "power:+5V") (at 144.78 137.16 180) (unit 1)
+    (in_bom yes) (on_board yes) (dnp no) (fields_autoplaced)
+    (property "Reference" "#PWR045" (at 144.78 133.35 0)
+      (effects (font (size 1.27 1.27)) hide)
+    )
+    (property "Value" "+5V" (at 144.78 142.24 0)
+      (effects (font (size 1.27 1.27)))
+    )
+    (property "Footprint" "" (at 144.78 137.16 0)
+      (effects (font (size 1.27 1.27)) hide)
+    )
+    (property "Datasheet" "" (at 144.78 137.16 0)
+      (effects (font (size 1.27 1.27)) hide)
+    )
+    (pin "1")
+    (instances
+      (project "fprpcb"
+        (path "/256b697e-9752-4e3a-a338-bc05701ab36e"
+          (reference "#PWR045") (unit 1)
+        )
+      )
+    )
+  )
   (symbol (lib_id "power:+3V3") (at 242.57 82.55 0) (unit 1)
     (in_bom yes) (on_board yes) (dnp no) (fields_autoplaced)
@@
         )
       )
+    )
+  )
+  (symbol (lib_id "power:+5V") (at 257.81 20.32 0) (unit 1)
+    (in_bom yes) (on_board yes) (dnp no)
+    (property "Reference" "#PWR032" (at 257.81 24.13 0)
+      (effects (font (size 1.27 1.27)) hide)
+    )
+    (property "Value" "VSYS" (at 258.445 17.145 0)
+      (effects (font (size 1.27 1.27)) (justify left))
+    )
+    (property "Footprint" "" (at 257.81 20.32 0)
+      (effects (font (size 1.27 1.27)) hide)
+    )
+    (property "Datasheet" "" (at 257.81 20.32 0)
+      (effects (font (size 1.27 1.27)) hide)
+    )
+    (pin "1")
+    (instances
+      (project "fprpcb"
+        (path "/256b697e-9752-4e3a-a338-bc05701ab36e"
+          (reference "#PWR032") (unit 1)
+        )
+      )
